File: oven-controller/eagle/oven-controller-v3.sch (EAGLE design)
At the start: 43 parts, among them Q1 FDV305N, Q2 FDV305N, Q3 FDV305N, Q4 FDV305N, U1 ARDUINO_SHIELDLONGPADS, U2 MAX31855, U3 MAX31855, U4 MAX31855, U5 MAX31855, U6 MAX31855

Commit message: Fixed FET resistors. Passes ERC, DRC. Needs review.
Parts:
- C1, C2, C3, C4, C5: value (none) -> 0.1u
Connections:
- removed net CS_LCD: U1.*D10
- removed net CS_SD: U1.D4
- removed net DC_LCD: U1.D8
- removed net JOY_READ: U1.A3
- removed net N$23: Q3.G, R10.1
- removed net RESET: U1.RX
- removed net SPI_MOSI: U1.*D11
- new net N$22: Q3.G, R10.1, R11.2
- net CS_FAN: no longer R11.2
- net CS_HEAT1: now also R5.2
- net CS_HEAT2: no longer R9.2
- net CS_VENT: no longer R2.2
- net N$2: now also R2.2
- net N$20: now also R9.2
Other:
- moved on the sheet: C1, C2, C3, C4, C5, FAN, HEAT1, HEAT2, LED1, LED2, LED3, LED4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
